Commit message: gz arm

File: src/my_robot_description/urdf/rubot_arm/rubot_mecanum_arm.urdf.xacro (robot description, xacro)
@@ -1,5 +1,5 @@
 <?xml version="1.0"?>
 <robot xmlns:xacro="http://ros.org/wiki/xacro" name="rubot_mecanum">
-  <xacro:include filename="$(find my_robot_description)/urdf/my_arm_mecanum_macro.xacro"/>
+  <xacro:include filename="$(find my_robot_description)/urdf/rubot_arm/my_arm_mecanum_macro.xacro"/>
     <material name="yellow">
         <color rgba="0.8 0.8 0.0 1.0"/>
@@ -17,11 +17,4 @@
         <color rgba="0.2 0.7 0.2 1.0"/>
     </material>
-  <!-- ===== Frames base ===== -->
-  <link name="base_footprint"/>
-  <joint name="base_link_joint" type="fixed">
-    <parent link="base_footprint"/>
-    <child link="base_link"/>
-    <origin xyz="0 0 0" rpy="0 0 0"/>
-  </joint>
   <link name="base_link">
     <!-- Visual (per RViz) -->
@@ -41,5 +34,24 @@
       </geometry>
     </collision>
+    <!-- Needed Inertia -->
+    <inertial>
+        <origin xyz="0 0 0.05" rpy="0 0 0"/>
+        <mass value="2.0"/>
+        <inertia
+            ixx="0.0142"
+            ixy="0.0"
+            ixz="0.0"
+            iyy="0.0217"
+            iyz="0.0"
+            izz="0.0308"/>
+    </inertial>
   </link>
+  <!-- ===== Frames base ===== -->
+  <link name="base_footprint"/>
+  <joint name="base_link_joint" type="fixed">
+    <parent link="base_link"/>
+    <child link="base_footprint"/>
+    <origin xyz="0 0 0" rpy="0 0 0"/>
+  </joint>
   <!-- ===== Rodes (només visuals, fixed) ===== -->
   <joint name="upper_left_wheel_joint" type="fixed">
@@ -133,5 +145,5 @@
     prefix="arm_"
     parent="base_link"
-    xyz="-0.10 0.00 0.12"
-    rpy="0 0 0"/>
+    xyz="-0.08 0.00 0.09"
+    rpy="0 0 3.14"/>
 </robot>

Commit message: ros2_control arm

File: src/my_robot_description/urdf/rubot_arm/rubot_mecanum_arm.urdf.xacro (robot description, xacro)
@@ -281,3 +281,47 @@
         </sensor>
     </gazebo>
+    <!-- =========================
+     ros2_control for SG90 arm in Gazebo
+     ========================= -->
+    <ros2_control name="ArmGazeboSystem" type="system">
+    <hardware>
+        <plugin>ign_ros2_control/IgnitionSystem</plugin>
+    </hardware>
+    <joint name="arm_joint1">
+        <command_interface name="position"/>
+        <state_interface name="position"/>
+        <state_interface name="velocity"/>
+    </joint>
+    <joint name="arm_joint2">
+        <command_interface name="position"/>
+        <state_interface name="position"/>
+        <state_interface name="velocity"/>
+    </joint>
+    <joint name="arm_joint3">
+        <command_interface name="position"/>
+        <state_interface name="position"/>
+        <state_interface name="velocity"/>
+    </joint>
+    <joint name="arm_joint4">
+        <command_interface name="position"/>
+        <state_interface name="position"/>
+        <state_interface name="velocity"/>
+    </joint>
+    <joint name="arm_joint5">
+        <command_interface name="position"/>
+        <state_interface name="position"/>
+        <state_interface name="velocity"/>
+    </joint>
+    <joint name="arm_joint6">
+        <command_interface name="position"/>
+        <state_interface name="position"/>
+        <state_interface name="velocity"/>
+    </joint>
+    </ros2_control>
+    <gazebo>
+    <plugin name="ign_ros2_control::IgnitionROS2ControlPlugin"
+            filename="libign_ros2_control-system.so">
+        <parameters>$(find my_robot_bringup)/config/arm_controllers.yaml</parameters>
+    </plugin>
+    </gazebo>
 </robot>
