Commit message: arm bringup

File: src/my_robot_description/urdf/rubot_arm/rubot_mecanum_arm.urdf.xacro (robot description, xacro)
@@ -27,4 +27,13 @@
         <color rgba="0.2 0.7 0.2 1.0"/>
     </material>
+    <material name="servo">
+      <color rgba="0.08 0.08 0.08 1.0"/>
+    </material>
+    <material name="metal">
+      <color rgba="0.45 0.45 0.45 1.0"/>
+    </material>
+    <material name="red">
+      <color rgba="0.80 0.05 0.05 1.0"/>
+    </material>
   <link name="base_link">
     <!-- Visual (per RViz) -->
@@ -60,6 +69,6 @@
   <link name="base_footprint"/>
   <joint name="base_link_joint" type="fixed">
-    <parent link="base_link"/>
-    <child link="base_footprint"/>
+    <parent link="base_footprint"/>
+    <child link="base_link"/>
     <origin xyz="0 0 0" rpy="0 0 0"/>
   </joint>

Commit message: updated yolo

File: src/my_robot_description/urdf/rubot_arm/rubot_mecanum_arm.urdf.xacro (robot description, xacro)
@@ -11,5 +11,5 @@
     xyz="-0.08 0.0 0.09"
     rpy="0 0 3.14159"
-    hardware_plugin="ign_ros2_control/IgnitionSystem"/>
+    hardware_plugin="$(arg hardware_plugin)"/>
     <material name="yellow">
         <color rgba="0.8 0.8 0.0 1.0"/>
@@ -36,4 +36,6 @@
       <color rgba="0.80 0.05 0.05 1.0"/>
     </material>
+  <!-- ===== Frames base ===== -->
+  <link name="base_footprint"/>
   <link name="base_link">
     <!-- Visual (per RViz) -->
@@ -66,7 +68,5 @@
     </inertial>
   </link>
-  <!-- ===== Frames base ===== -->
-  <link name="base_footprint"/>
-  <joint name="base_link_joint" type="fixed">
+  <joint name="base_footprint_joint" type="fixed">
     <parent link="base_footprint"/>
     <child link="base_link"/>
@@ -237,5 +237,5 @@
             name="ignition::gazebo::systems::OdometryPublisher">
         <odom_frame>odom</odom_frame>
-        <robot_base_frame>base_link</robot_base_frame>
+        <robot_base_frame>base_footprint</robot_base_frame>
         <odom_topic>/odom</odom_topic>
         <tf_topic>/tf</tf_topic>
