Commit message: bringup arm

File: src/my_robot_description/urdf/rubot_arm/my_arm_mecanum_macro.xacro (robot description, xacro)
@@ -284,4 +284,28 @@
         oz="0"/>
     </link>
+    <gazebo reference="${prefix}arm_base_link">
+    <gravity>false</gravity>
+    </gazebo>
+    <gazebo reference="${prefix}link1">
+    <gravity>false</gravity>
+    </gazebo>
+    <gazebo reference="${prefix}link2">
+    <gravity>false</gravity>
+    </gazebo>
+    <gazebo reference="${prefix}link3">
+    <gravity>false</gravity>
+    </gazebo>
+    <gazebo reference="${prefix}link4">
+    <gravity>false</gravity>
+    </gazebo>
+    <gazebo reference="${prefix}link5">
+    <gravity>false</gravity>
+    </gazebo>
+    <gazebo reference="${prefix}link6">
+    <gravity>false</gravity>
+    </gazebo>
+    <gazebo reference="${prefix}link6_right">
+    <gravity>false</gravity>
+    </gazebo>
   </xacro:macro>
 </robot>

File: src/my_robot_description/urdf/rubot_arm/rubot_mecanum_arm.urdf.xacro (robot description, xacro)
@@ -68,4 +68,20 @@
       <material name="light_grey"/>
     </visual>
+    <collision>
+        <origin xyz="0 0 0" rpy="1.5708 0 0"/>
+        <geometry>
+            <cylinder radius="0.04" length="0.035"/>
+        </geometry>
+    </collision>
+    <inertial>
+        <mass value="0.05"/>
+        <inertia
+            ixx="0.00003"
+            ixy="0.0"
+            ixz="0.0"
+            iyy="0.00003"
+            iyz="0.0"
+            izz="0.00004"/>
+    </inertial>
   </link>
   <joint name="lower_left_wheel_joint" type="fixed">
@@ -82,4 +98,20 @@
       <material name="light_grey"/>
     </visual>
+    <collision>
+        <origin xyz="0 0 0" rpy="1.5708 0 0"/>
+        <geometry>
+            <cylinder radius="0.04" length="0.035"/>
+        </geometry>
+    </collision>
+    <inertial>
+        <mass value="0.05"/>
+        <inertia
+            ixx="0.00003"
+            ixy="0.0"
+            ixz="0.0"
+            iyy="0.00003"
+            iyz="0.0"
+            izz="0.00004"/>
+    </inertial>
   </link>
   <joint name="upper_right_wheel_joint" type="fixed">
@@ -96,4 +128,20 @@
       <material name="light_grey"/>
     </visual>
+    <collision>
+        <origin xyz="0 0 0" rpy="1.5708 0 0"/>
+        <geometry>
+            <cylinder radius="0.04" length="0.035"/>
+        </geometry>
+    </collision>
+    <inertial>
+        <mass value="0.05"/>
+        <inertia
+            ixx="0.00003"
+            ixy="0.0"
+            ixz="0.0"
+            iyy="0.00003"
+            iyz="0.0"
+            izz="0.00004"/>
+    </inertial>
   </link>
   <joint name="lower_right_wheel_joint" type="fixed">
@@ -110,4 +158,20 @@
       <material name="light_grey"/>
     </visual>
+    <collision>
+        <origin xyz="0 0 0" rpy="1.5708 0 0"/>
+        <geometry>
+            <cylinder radius="0.04" length="0.035"/>
+        </geometry>
+    </collision>
+    <inertial>
+        <mass value="0.05"/>
+        <inertia
+            ixx="0.00003"
+            ixy="0.0"
+            ixz="0.0"
+            iyy="0.00003"
+            iyz="0.0"
+            izz="0.00004"/>
+    </inertial>
   </link>
   <!-- ===== Lidar frame ===== -->
@@ -147,3 +211,73 @@
     xyz="-0.08 0.00 0.09"
     rpy="0 0 3.14"/>
+    <!-- =========================
+        Gazebo plugins
+        ========================= -->
+    <gazebo>
+    <!-- Holonomic / planar velocity control -->
+    <plugin filename="libignition-gazebo6-velocity-control-system.so"
+            name="ignition::gazebo::systems::VelocityControl">
+        <topic>/cmd_vel</topic>
+    </plugin>
+    <!-- Odometry publisher -->
+    <plugin filename="libignition-gazebo6-odometry-publisher-system.so"
+            name="ignition::gazebo::systems::OdometryPublisher">
+        <odom_frame>odom</odom_frame>
+        <robot_base_frame>base_link</robot_base_frame>
+        <odom_topic>/odom</odom_topic>
+        <tf_topic>/tf</tf_topic>
+        <odom_publish_frequency>50</odom_publish_frequency>
+    </plugin>
+    </gazebo>
+    <!-- =========================
+     Gazebo lidar sensor
+     ========================= -->
+    <gazebo reference="base_scan">
+        <sensor name="lidar" type="gpu_lidar">
+            <pose>0 0 0 0 0 0</pose>
+            <topic>/scan</topic>
+            <update_rate>10</update_rate>
+            <ray>
+            <scan>
+                <horizontal>
+                <samples>360</samples>
+                <resolution>1</resolution>
+                <min_angle>-3.14159</min_angle>
+                <max_angle>3.14159</max_angle>
+                </horizontal>
+            </scan>
+            <range>
+                <min>0.12</min>
+                <max>10.0</max>
+                <resolution>0.01</resolution>
+            </range>
+            </ray>
+            <always_on>true</always_on>
+            <visualize>true</visualize>
+        </sensor>
+    </gazebo>
+    <!-- =========================
+        Gazebo RGBD camera sensor
+        ========================= -->
+    <gazebo reference="camera">
+        <sensor name="rgbd_camera" type="rgbd_camera">
+            <pose>0 0 0 0 0 0</pose>
+            <topic>/camera</topic>
+            <update_rate>15</update_rate>
+            <camera>
+            <horizontal_fov>1.047</horizontal_fov>
+            <image>
+                <width>640</width>
+                <height>480</height>
+                <format>R8G8B8</format>
+            </image>
+            <clip>
+                <near>0.05</near>
+                <far>10.0</far>
+            </clip>
+            </camera>
+            <always_on>true</always_on>
+            <visualize>true</visualize>
+        </sensor>
+    </gazebo>
 </robot>

Commit message: wallfollower

File: src/my_robot_description/urdf/rubot_arm/my_arm_mecanum_macro.xacro (robot description, xacro)
@@ -284,28 +284,64 @@
         oz="0"/>
     </link>
-    <gazebo reference="${prefix}arm_base_link">
-    <gravity>false</gravity>
-    </gazebo>
-    <gazebo reference="${prefix}link1">
-    <gravity>false</gravity>
-    </gazebo>
-    <gazebo reference="${prefix}link2">
-    <gravity>false</gravity>
-    </gazebo>
-    <gazebo reference="${prefix}link3">
-    <gravity>false</gravity>
-    </gazebo>
-    <gazebo reference="${prefix}link4">
-    <gravity>false</gravity>
-    </gazebo>
-    <gazebo reference="${prefix}link5">
-    <gravity>false</gravity>
-    </gazebo>
-    <gazebo reference="${prefix}link6">
-    <gravity>false</gravity>
-    </gazebo>
-    <gazebo reference="${prefix}link6_right">
-    <gravity>false</gravity>
-    </gazebo>
+    <link name="${prefix}tool">
+    <visual>
+        <origin xyz="0 0 0" rpy="0 0 0"/>
+        <geometry>
+        <sphere radius="0.008"/>
+        </geometry>
+        <material name="black"/>
+    </visual>
+    <collision>
+        <geometry>
+        <sphere radius="0.008"/>
+        </geometry>
+    </collision>
+    </link>
+    <joint name="${prefix}link5_to_tool" type="fixed">
+        <parent link="${prefix}link5"/>
+        <child link="${prefix}tool"/>
+        <origin xyz="0.050 0 0" rpy="0 0 0"/>
+    </joint>
+    <ros2_control name="${prefix}RubotMecanumArmSystem" type="system">
+        <hardware>
+            <plugin>$(arg hardware_plugin)</plugin>
+        </hardware>
+        <joint name="${prefix}joint1">
+            <param name="position_proportional_gain">5.0</param>
+            <command_interface name="position"/>
+            <state_interface name="position"/>
+            <state_interface name="velocity"/>
+        </joint>
+        <joint name="${prefix}joint2">
+            <param name="position_proportional_gain">5.0</param>
+            <command_interface name="position"/>
+            <state_interface name="position"/>
+            <state_interface name="velocity"/>
+        </joint>
+        <joint name="${prefix}joint3">
+            <param name="position_proportional_gain">5.0</param>
+            <command_interface name="position"/>
+            <state_interface name="position"/>
+            <state_interface name="velocity"/>
+        </joint>
+        <joint name="${prefix}joint4">
+            <param name="position_proportional_gain">5.0</param>
+            <command_interface name="position"/>
+            <state_interface name="position"/>
+            <state_interface name="velocity"/>
+        </joint>
+        <joint name="${prefix}joint5">
+            <param name="position_proportional_gain">5.0</param>
+            <command_interface name="position"/>
+            <state_interface name="position"/>
+            <state_interface name="velocity"/>
+        </joint>
+        <joint name="${prefix}joint6">
+            <param name="position_proportional_gain">5.0</param>
+            <command_interface name="position"/>
+            <state_interface name="position"/>
+            <state_interface name="velocity"/>
+        </joint>
+    </ros2_control>
   </xacro:macro>
 </robot>

File: src/my_robot_description/urdf/rubot_arm/rubot_mecanum_arm.urdf.xacro (robot description, xacro)
@@ -1,4 +1,8 @@
 <?xml version="1.0"?>
 <robot xmlns:xacro="http://ros.org/wiki/xacro" name="rubot_mecanum">
+    <!-- ros2_control arguments -->
+    <xacro:arg name="use_gazebo_plugin" default="true"/>
+    <xacro:arg name="hardware_plugin" default="ign_ros2_control/IgnitionSystem"/>
+    <xacro:arg name="ros2_control_params" default=""/>
   <xacro:include filename="$(find my_robot_description)/urdf/rubot_arm/my_arm_mecanum_macro.xacro"/>
     <material name="yellow">
@@ -254,5 +258,5 @@
             </ray>
             <always_on>true</always_on>
-            <visualize>true</visualize>
+            <visualize>false</visualize>
         </sensor>
     </gazebo>
@@ -268,6 +272,6 @@
             <horizontal_fov>1.047</horizontal_fov>
             <image>
-                <width>640</width>
-                <height>480</height>
+                <width>320</width>
+                <height>240</height>
                 <format>R8G8B8</format>
             </image>
@@ -278,50 +282,15 @@
             </camera>
             <always_on>true</always_on>
-            <visualize>true</visualize>
+            <visualize>false</visualize>
         </sensor>
     </gazebo>
-    <!-- =========================
-     ros2_control for SG90 arm in Gazebo
-     ========================= -->
-    <ros2_control name="ArmGazeboSystem" type="system">
-    <hardware>
-        <plugin>ign_ros2_control/IgnitionSystem</plugin>
-    </hardware>
-    <joint name="arm_joint1">
-        <command_interface name="position"/>
-        <state_interface name="position"/>
-        <state_interface name="velocity"/>
-    </joint>
-    <joint name="arm_joint2">
-        <command_interface name="position"/>
-        <state_interface name="position"/>
-        <state_interface name="velocity"/>
-    </joint>
-    <joint name="arm_joint3">
-        <command_interface name="position"/>
-        <state_interface name="position"/>
-        <state_interface name="velocity"/>
-    </joint>
-    <joint name="arm_joint4">
-        <command_interface name="position"/>
-        <state_interface name="position"/>
-        <state_interface name="velocity"/>
-    </joint>
-    <joint name="arm_joint5">
-        <command_interface name="position"/>
-        <state_interface name="position"/>
-        <state_interface name="velocity"/>
-    </joint>
-    <joint name="arm_joint6">
-        <command_interface name="position"/>
-        <state_interface name="position"/>
-        <state_interface name="velocity"/>
-    </joint>
-    </ros2_control>
-    <gazebo>
-    <plugin name="ign_ros2_control::IgnitionROS2ControlPlugin"
+    <xacro:if value="$(arg use_gazebo_plugin)">
+        <gazebo>
+            <plugin
+            name="ign_ros2_control::IgnitionROS2ControlPlugin"
             filename="libign_ros2_control-system.so">
-        <parameters>$(find my_robot_bringup)/config/arm_controllers.yaml</parameters>
-    </plugin>
-    </gazebo>
+            <parameters>$(arg ros2_control_params)</parameters>
+            </plugin>
+        </gazebo>
+    </xacro:if>
 </robot>

Commit message: params

File: src/my_robot_description/urdf/rubot_arm/my_arm_mecanum_macro.xacro (robot description, xacro)
@@ -65,5 +65,5 @@
       </collision>
       <xacro:inertial_box
-        mass="0.08"
+        mass="0.008"
         x="0.08"
         y="0.08"
@@ -96,5 +96,5 @@
       </collision>
       <xacro:inertial_cylinder_z
-        mass="0.03"
+        mass="0.003"
         radius="0.012"
         length="0.055"
@@ -126,5 +126,5 @@
       </collision>
       <xacro:inertial_cylinder_x
-        mass="0.025"
+        mass="0.0025"
         radius="0.012"
         length="0.075"
@@ -156,5 +156,5 @@
       </collision>
       <xacro:inertial_cylinder_x
-        mass="0.025"
+        mass="0.0025"
         radius="0.012"
         length="0.075"
@@ -186,5 +186,5 @@
       </collision>
       <xacro:inertial_cylinder_x
-        mass="0.015"
+        mass="0.0015"
         radius="0.010"
         length="0.045"
@@ -216,5 +216,5 @@
       </collision>
       <xacro:inertial_box
-        mass="0.02"
+        mass="0.002"
         x="0.030"
         y="0.030"
@@ -247,5 +247,5 @@
     </collision>
     <xacro:inertial_box
-        mass="0.005"
+        mass="0.0005"
         x="0.050"
         y="0.008"
@@ -276,5 +276,5 @@
     </collision>
     <xacro:inertial_box
-        mass="0.005"
+        mass="0.0005"
         x="0.050"
         y="0.008"
@@ -344,4 +344,25 @@
         </joint>
     </ros2_control>
+    <gazebo reference="${prefix}arm_base_link">
+        <gravity>false</gravity>
+    </gazebo>
+    <gazebo reference="${prefix}link1">
+        <gravity>false</gravity>
+    </gazebo>
+    <gazebo reference="${prefix}link2">
+        <gravity>false</gravity>
+    </gazebo>
+    <gazebo reference="${prefix}link3">
+        <gravity>false</gravity>
+    </gazebo>
+    <gazebo reference="${prefix}link4">
+        <gravity>false</gravity>
+    </gazebo>
+    <gazebo reference="${prefix}link5">
+        <gravity>false</gravity>
+    </gazebo>
+    <gazebo reference="${prefix}link6">
+        <gravity>false</gravity>
+    </gazebo>
   </xacro:macro>
 </robot>

File: src/my_robot_description/urdf/rubot_arm/rubot_mecanum_arm.urdf.xacro (robot description, xacro)
@@ -40,13 +40,13 @@
     <!-- Needed Inertia -->
     <inertial>
-        <origin xyz="0 0 0.05" rpy="0 0 0"/>
-        <mass value="2.0"/>
-        <inertia
-            ixx="0.0142"
-            ixy="0.0"
-            ixz="0.0"
-            iyy="0.0217"
-            iyz="0.0"
-            izz="0.0308"/>
+        <origin xyz="0 0 0.02" rpy="0 0 0"/>
+        <mass value="3.0"/>
+        <inertia
+            ixx="0.03"
+            ixy="0.0"
+            ixz="0.0"
+            iyy="0.08"
+            iyz="0.0"
+            izz="0.05"/>
     </inertial>
   </link>
@@ -247,6 +247,6 @@
                 <samples>360</samples>
                 <resolution>1</resolution>
-                <min_angle>-3.14159</min_angle>
-                <max_angle>3.14159</max_angle>
+                <min_angle>-2.3</min_angle>
+                <max_angle>2.3</max_angle>
                 </horizontal>
             </scan>
