Commit message: arm corrections

File: src/my_robot_description/urdf/rubot_arm/my_arm_mecanum_macro.xacro (robot description, xacro)
@@ -45,10 +45,10 @@
   <xacro:macro name="my_arm_mecanum" params="prefix parent xyz rpy">
     <!-- Mount joint: robot base_link -> arm base -->
-    <joint name="${prefix}arm_mount_joint" type="fixed">
+    <joint name="${prefix}mount_joint" type="fixed">
       <parent link="${parent}"/>
-      <child link="${prefix}arm_base_link"/>
+      <child link="${prefix}base_link"/>
       <origin xyz="${xyz}" rpy="${rpy}"/>
     </joint>
-    <link name="${prefix}arm_base_link">
+    <link name="${prefix}base_link">
       <visual>
         <origin xyz="0 0 0.015" rpy="0 0 0"/>
@@ -75,5 +75,5 @@
     <!-- joint1: base yaw -->
     <joint name="${prefix}joint1" type="revolute">
-      <parent link="${prefix}arm_base_link"/>
+      <parent link="${prefix}base_link"/>
       <child link="${prefix}link1"/>
       <origin xyz="0 0 0.03" rpy="0 0 0"/>
@@ -344,5 +344,5 @@
         </joint>
     </ros2_control>
-    <gazebo reference="${prefix}arm_base_link">
+    <gazebo reference="${prefix}base_link">
         <gravity>false</gravity>
     </gazebo>
