Commit message: updated model

File: src/my_robot_description/urdf/rubot/rubot_mecanum.urdf.xacro (robot description, xacro)
@@ -20,4 +20,6 @@
         <color rgba="0.2 0.7 0.2 1.0"/>
     </material>
+<!-- ===== Frames base ===== -->
+  <link name="base_footprint"/>
   <link name="base_link">
     <!-- Visual (per RViz) -->
@@ -50,9 +52,7 @@
     </inertial>
   </link>
-  <!-- ===== Frames base ===== -->
-  <link name="base_footprint"/>
-  <joint name="base_link_joint" type="fixed">
-    <parent link="base_link"/>
-    <child link="base_footprint"/>
+  <joint name="base_footprint_joint" type="fixed">
+    <parent link="base_footprint"/>
+    <child link="base_link"/>
     <origin xyz="0 0 0" rpy="0 0 0"/>
   </joint>
@@ -221,5 +221,5 @@
             name="ignition::gazebo::systems::OdometryPublisher">
         <odom_frame>odom</odom_frame>
-        <robot_base_frame>base_link</robot_base_frame>
+        <robot_base_frame>base_footprint</robot_base_frame>
         <odom_topic>/odom</odom_topic>
         <tf_topic>/tf</tf_topic>
